File: pidaqv2.kicad_pcb (KiCad board)
At the start: 2 copper layers, 26 parts, among them J101 Screw_Terminal_01x10, J102 Screw_Terminal_01x06, J103 Conn_01x02_Male, J104 Screw_Terminal_01x04, J105 Screw_Terminal_01x08, U201 ADS1261BIRHBR, U301 ADS1261BIRHBR, U401 AD8426ACPZ-R7

Commit message: temporarily complete
Routing:
- net GND: track 56.0 -> 46.9 mm, vias 13 -> 17
Changed lines of the file:
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@@
     (thickness 1.6)
     (drawings 0)
-    (tracks 390)
+    (tracks 381)
     (zones 0)
     (modules 26)
@@
   (segment (start 164.3072 104.3931) (end 164.3072 104.796174) (width 0.1778) (layer F.Cu) (net 1))
   (segment (start 160.542 106.553) (end 160.542 106.553) (width 0.1778) (layer F.Cu) (net 1))
-  (segment (start 166.6062 94.0816) (end 167.0812 94.0816) (width 0.1778) (layer F.Cu) (net 1))
-  (segment (start 165.3072 95.3806) (end 166.6062 94.0816) (width 0.1778) (layer F.Cu) (net 1))
   (segment (start 165.3072 99.5181) (end 165.3072 95.3806) (width 0.1778) (layer F.Cu) (net 1))
-  (segment (start 164.8892 94.0956) (end 164.4142 94.0956) (width 0.1778) (layer F.Cu) (net 1))
-  (segment (start 165.3072 94.5136) (end 164.8892 94.0956) (width 0.1778) (layer F.Cu) (net 1))
-  (segment (start 165.3072 95.3806) (end 165.3072 94.5136) (width 0.1778) (layer F.Cu) (net 1))
   (segment (start 164.4142 94.0956) (end 164.4142 94.0956) (width 0.1778) (layer F.Cu) (net 1))
-  (via (at 164.4142 94.0956) (size 0.8) (drill 0.4) (layers F.Cu B.Cu) (net 1))
   (segment (start 164.3072 104.3931) (end 164.3389 104.3931) (width 0.1778) (layer F.Cu) (net 1))
   (segment (start 136.4234 87.66) (end 136.4459 87.6375) (width 0.1778) (layer F.Cu) (net 1))
@@
   (segment (start 139.954 87.66) (end 139.9315 87.6375) (width 0.1778) (layer F.Cu) (net 1))
   (segment (start 168.8592 94.1096) (end 168.8592 94.1096) (width 0.1778) (layer F.Cu) (net 1))
-  (segment (start 167.0812 94.0816) (end 168.8312 94.0816) (width 0.1778) (layer F.Cu) (net 1))
   (segment (start 168.8312 94.0816) (end 168.8592 94.1096) (width 0.1778) (layer F.Cu) (net 1))
-  (via (at 168.8592 94.1096) (size 0.8) (drill 0.4) (layers F.Cu B.Cu) (net 1))
   (segment (start 160.542 106.553) (end 160.542 106.553) (width 0.1778) (layer F.Cu) (net 1))
   (segment (start 162.9947 103.8306) (end 162.8059 103.8306) (width 0.1778) (layer F.Cu) (net 1))
@@
   (segment (start 139.954 87.010002) (end 140.6652 87.010002) (width 0.1778) (layer F.Cu) (net 40))
   (segment (start 140.5074 100.5024) (end 140.5074 101.3469) (width 0.1778) (layer F.Cu) (net 41))
-  (segment (start 140.6144 111.7574) (end 139.5121 111.7574) (width 0.1778) (layer F.Cu) (net 1))
+  (segment (start 140.6144 111.7574) (end 138.4554 111.7574) (width 0.1778) (layer F.Cu) (net 1))
   (segment (start 143.0274 111.7574) (end 143.0274 111.7574) (width 0.1778) (layer F.Cu) (net 1))
-  (segment (start 165.3072 101.7056) (end 165.5572 101.9556) (width 0.1778) (layer F.Cu) (net 1))
   (segment (start 162.2425 104.394) (end 162.2425 104.394) (width 0.1778) (layer F.Cu) (net 1))
   (via (at 145.4404 100.6856) (size 0.8) (drill 0.4) (layers F.Cu B.Cu) (net 1))
@@
   (segment (start 162.6822 100.2056) (end 160.7185 98.2419) (width 0.1778) (layer F.Cu) (net 1))
   (via (at 162.2425 104.394) (size 0.8) (drill 0.4) (layers F.Cu B.Cu) (net 1))
+  (segment (start 166.6062 94.0816) (end 167.0812 94.0816) (width 0.1778) (layer F.Cu) (net 1))
+  (via (at 168.8592 94.1096) (size 0.8) (drill 0.4) (layers F.Cu B.Cu) (net 1))
+  (segment (start 167.0812 94.0816) (end 168.8312 94.0816) (width 0.1778) (layer F.Cu) (net 1))
+  (via (at 164.4142 94.0956) (size 0.8) (drill 0.4) (layers F.Cu B.Cu) (net 1))
+  (segment (start 164.8892 94.0956) (end 164.4142 94.0956) (width 0.1778) (layer F.Cu) (net 1))
+  (segment (start 165.3072 94.5136) (end 164.8892 94.0956) (width 0.1778) (layer F.Cu) (net 1))
+  (segment (start 165.3072 95.3806) (end 165.3072 94.5136) (width 0.1778) (layer F.Cu) (net 1))
+  (segment (start 165.3072 95.3806) (end 166.6062 94.0816) (width 0.1778) (layer F.Cu) (net 1))
+  (via (at 159.385 103.251) (size 0.8) (drill 0.4) (layers F.Cu B.Cu) (net 1))
+  (via (at 160.542 106.553) (size 0.8) (drill 0.4) (layers F.Cu B.Cu) (net 1) (status 1000000))
+  (segment (start 143.0274 111.7574) (end 142.5524 111.7574) (width 0.1778) (layer F.Cu) (net 1))
+  (segment (start 141.0894 111.7574) (end 140.6144 111.7574) (width 0.1778) (layer F.Cu) (net 1))
+  (segment (start 142.5524 111.7574) (end 142.0074 111.2124) (width 0.1778) (layer F.Cu) (net 1))
+  (segment (start 142.0074 111.2124) (end 142.0074 110.8394) (width 0.1778) (layer F.Cu) (net 1))
+  (segment (start 142.0074 106.2219) (end 142.0074 110.8394) (width 0.1778) (layer F.Cu) (net 1))
+  (segment (start 142.0074 110.8394) (end 141.0894 111.7574) (width 0.1778) (layer F.Cu) (net 1))
+  (via (at 143.0274 111.7574) (size 0.8) (drill 0.4) (layers F.Cu B.Cu) (net 1))
+  (via (at 140.6144 111.7574) (size 0.8) (drill 0.4) (layers F.Cu B.Cu) (net 1) (status 1000000))
+  (via (at 138.4554 111.7574) (size 0.8) (drill 0.4) (layers F.Cu B.Cu) (net 1))
+  (via (at 148.717 101.727) (size 0.8) (drill 0.4) (layers F.Cu B.Cu) (net 1))
+  (via (at 141.7854 99.3394) (size 0.8) (drill 0.4) (layers F.Cu B.Cu) (net 1))
+  (via (at 132.588 85.344) (size 0.8) (drill 0.4) (layers F.Cu B.Cu) (net 1))
+  (via (at 132.6515 87.122) (size 0.8) (drill 0.4) (layers F.Cu B.Cu) (net 1))
   (segment (start 132.616 87.122) (end 132.6515 87.122) (width 0.1778) (layer F.Cu) (net 1))
-  (via (at 132.588 88.646) (size 0.8) (drill 0.4) (layers F.Cu B.Cu) (net 1))
-  (segment (start 132.588 85.344) (end 132.588 88.646) (width 0.1778) (layer F.Cu) (net 1))
-  (via (at 142.5575 97.79) (size 0.8) (drill 0.4) (layers F.Cu B.Cu) (net 1))
-  (segment (start 141.7854 99.3394) (end 141.7854 98.5621) (width 0.1778) (layer F.Cu) (net 1))
-  (segment (start 141.7854 98.5621) (end 142.5575 97.79) (width 0.1778) (layer F.Cu) (net 1))
-  (via (at 149.606 100.33) (size 0.8) (drill 0.4) (layers F.Cu B.Cu) (net 1))
-  (segment (start 149.606 101.3223) (end 149.606 100.33) (width 0.1778) (layer F.Cu) (net 1))
-  (segment (start 148.7144 101.6889) (end 149.2394 101.6889) (width 0.1778) (layer F.Cu) (net 1))
-  (segment (start 149.2394 101.6889) (end 149.606 101.3223) (width 0.1778) (layer F.Cu) (net 1))
-  (segment (start 139.5121 111.7574) (end 138.4554 111.7574) (width 0.1778) (layer F.Cu) (net 1))
-  (via (at 141.7955 110.871) (size 0.8) (drill 0.4) (layers F.Cu B.Cu) (net 1))
-  (segment (start 142.0074 106.2219) (end 142.0074 110.6591) (width 0.1778) (layer F.Cu) (net 1))
-  (segment (start 142.0074 110.6591) (end 141.7955 110.871) (width 0.1778) (layer F.Cu) (net 1))
-  (segment (start 141.474785 111.7574) (end 141.0894 111.7574) (width 0.1778) (layer F.Cu) (net 1))
-  (segment (start 141.0894 111.7574) (end 140.6144 111.7574) (width 0.1778) (layer F.Cu) (net 1))
-  (segment (start 141.7955 111.436685) (end 141.474785 111.7574) (width 0.1778) (layer F.Cu) (net 1))
-  (segment (start 142.5524 111.7574) (end 143.0274 111.7574) (width 0.1778) (layer F.Cu) (net 1))
-  (segment (start 142.116215 111.7574) (end 142.5524 111.7574) (width 0.1778) (layer F.Cu) (net 1))
-  (segment (start 141.7955 111.436685) (end 142.116215 111.7574) (width 0.1778) (layer F.Cu) (net 1))
-  (segment (start 141.7955 110.871) (end 141.7955 111.436685) (width 0.1778) (layer F.Cu) (net 1))
-  (segment (start 159.3495 105.8855) (end 160.017 106.553) (width 0.1778) (layer F.Cu) (net 1))
-  (segment (start 160.017 106.553) (end 160.542 106.553) (width 0.1778) (layer F.Cu) (net 1))
-  (segment (start 159.3495 103.2256) (end 159.3495 105.255) (width 0.1778) (layer F.Cu) (net 1))
-  (segment (start 159.3495 105.255) (end 159.3495 105.8855) (width 0.1778) (layer F.Cu) (net 1))
-  (via (at 159.3495 105.255) (size 0.8) (drill 0.4) (layers F.Cu B.Cu) (net 1))
+  (segment (start 165.3072 101.7056) (end 165.5572 101.9556) (width 0.1778) (layer F.Cu) (net 1))
+  (segment (start 165.3072 99.5181) (end 165.3072 101.7056) (width 0.1778) (layer F.Cu) (net 1))
   (via (at 162.292 106.553) (size 0.8) (drill 0.4) (layers F.Cu B.Cu) (net 7))
   (segment (start 161.417 99.1235) (end 162.6235 97.917) (width 0.1778) (layer B.Cu) (net 7))
